File: Resources/PCB/V3.8/einkPDA_keyboard/einkPDA_keyboard.kicad_pcb (KiCad board)
At the start: 4 copper layers, 95 x 55.5 mm, 158 parts, among them J1 USB_C_Receptacle_USB2.0_16P, J2 Conn_01x12_Pin, J3 Conn_01x26_Pin, J4 Micro_SD_Card, J5 Conn_01x12_Pin, J6 C2764211, Q1 MMBT3904, Q2 AO3401A, SW36 YTS-C017-2B, SW4 SW_DIP_x02, SW41 YTS-C017-2B, U1 ESP32-S3-WROOM-1-N16R2, U10 TS3USB30ERSWR, U2 USBLC6-2SC6, U3 TPS63001, U4 PCF8563T, U5 TCA8418RTWR, U6 USBLC6-2SC6, U7 TPS61040DBV, U8 TPS22917DBV, U9 MP2722GRH-0000-Z, Y1 Crystal_32.768kHz

Commit message: PCB updates
Parts:
- F1: value 10A FUSE -> 3A FUSE
- moved TP7 28.6 mm to (125.9, 72.4)
- moved TP9 7.68 mm to (139.3, 71.0)
- moved TP8 7.19 mm to (140.2, 72.9)
- moved TP12 4.78 mm to (114.3, 74.0)
- moved TP6 2.68 mm to (86.4, 64.7)
- moved TP4 1.40 mm to (86.4, 62.6)
Connections:
- REF** pad : GND -> (no net) (x3)
Routing:
- net I2C_SCL: track 194.7 -> 180.6 mm, vias 10 -> 9
- net I2C_SDA: track 186.1 -> 181.1 mm, vias 8 -> 7
- net +12V: track 50.5 -> 46.8 mm
- net I2C_SDA_SWITCHED: track 157.6 -> 154.5 mm
- net V_LOADSWITCH: track 225.4 -> 223.5 mm, vias 11 -> 10
- net +3.3V: track 369.1 -> 367.5 mm
Other:
- board text added: "@Ashtf // V3.9"
- board text removed: "@Ashtf // V3.7"
