File: Resources/PCB/V3.8/einkPDA_keyboard/einkPDA_keyboard.kicad_sch (KiCad schematic)
At the start: 148 parts, among them J1 USB_C_Receptacle_USB2.0_16P, J2 Conn_01x12_Pin, J3 Conn_01x26_Pin, J4 Micro_SD_Card, J5 Conn_01x12_Pin, J6 C2764211, Q1 MMBT3904, Q2 AO3401A, SW36 YTS-C017-2B, SW4 SW_DIP_x02, SW41 YTS-C017-2B, U1 ESP32-S3-WROOM-1-N16R2, U10 TS3USB30ERSWR, U2 USBLC6-2SC6, U3 TPS63001, U4 PCF8563T, U5 TCA8418RTWR, U6 USBLC6-2SC6, U7 TPS61040DBV, U8 TPS22917DBV, U9 MP2722GRH-0000-Z, Y1 Crystal_32.768kHz

Commit message: PCB updates
Parts:
- F1: value 10A FUSE -> 3A FUSE; LCSC Part # C2760308 -> C2843999
Changed lines of the file:
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@@
 			)
 		)
-		(property "Value" "10A FUSE"
+		(property "Value" "3A FUSE"
 			(at 63.246 215.392 90)
 			(effects
@@
 			)
 		)
-		(property "LCSC Part #" "C2760308 "
+		(property "LCSC Part #" "C2843999"
 			(at 69.85 210.82 0)
 			(effects
