File: Resources/PCB/V3.8/einkPDA_screen/einkPDA_screen.kicad_pcb (KiCad board)
At the start: 2 copper layers, 95 x 54 mm, 47 parts, among them J1 Conn_01x12_Pin, J4 Conn_01x12_Pin, Q1 Si1308EDL, U1 MPR121QR2, U2 TPD4E02B04DQA, U3 TPD4E02B04DQA, U4 TPD4E02B04DQA

Commit message: PCB updates
Other:
- board text added: "@Ashtf // V3.9"
- board text removed: "@Ashtf // V3.8"
Changed lines of the file:
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@@
 		)
 	)
-	(gr_text "@Ashtf // V3.8"
+	(gr_text "@Ashtf // V3.9"
 		(at 113.05 129.875 0)
 		(layer "B.SilkS")
@@
 			(justify left bottom mirror)
 		)
-		(render_cache "@Ashtf // V3.8" 0
+		(render_cache "@Ashtf // V3.9" 0
 			(polygon
 				(pts
@@
 			(polygon
 				(pts
-					(xy 97.644062 127.835647) (xy 97.737055 127.855982) (xy 97.811551 127.886971) (xy 97.879926 127.932067)
-					(xy 97.93263 127.983792) (xy 97.971942 128.042309) (xy 98.010602 128.142376) (xy 98.02334 128.24784)
-					(xy 98.017352 128.326321) (xy 98.000372 128.392771) (xy 97.973118 128.449462) (xy 97.93524 128.498273)
-					(xy 97.875748 128.552091) (xy 97.788256 128.611639) (xy 97.736858 128.642414) (xy 97.850242 128.713523)
-					(xy 97.938273 128.783021) (xy 98.004961 128.850875) (xy 98.057192 128.930047) (xy 98.088437 129.019879)
-					(xy 98.099208 129.123695) (xy 98.089361 129.229073) (xy 98.061409 129.316702) (xy 98.015933 129.390413)
-					(xy 97.951105 129.452445) (xy 97.848088 129.511679) (xy 97.722872 129.549424) (xy 97.570376 129.562965)
-					(xy 97.444339 129.553645) (xy 97.340337 129.52774) (xy 97.254616 129.487494) (xy 97.176001 129.43084)
-					(xy 97.114739 129.36793) (xy 97.068473 129.298572) (xy 97.033353 129.220763) (xy 97.013577 129.148016)
-					(xy 97.012378 129.13493) (xy 97.310823 129.13493) (xy 97.316326 129.22362) (xy 97.330905 129.288957)
-					(xy 97.352496 129.336308) (xy 97.399275 129.393457) (xy 97.452834 129.427288) (xy 97.511404 129.445364)
-					(xy 97.565461 129.451102) (xy 97.63273 129.442063) (xy 97.688141 129.416365) (xy 97.734401 129.374166)
-					(xy 97.766745 129.31759) (xy 97.789275 129.230558) (xy 97.798087 129.101346) (xy 97.789538 128.985209)
-					(xy 97.775008 128.916911) (xy 97.746689 128.842449) (xy 97.703652 128.773519) (xy 97.63652 128.706772)
-					(xy 97.504232 128.787861) (xy 97.423948 128.844685) (xy 97.374616 128.895694) (xy 97.340003 128.952571)
-					(xy 97.321936 129.009023) (xy 97.310823 129.13493) (xy 97.012378 129.13493) (xy 97.007244 129.078876)
-					(xy 97.019674 128.958479) (xy 97.057466 128.841106) (xy 97.096732 128.770441) (xy 97.148832 128.709124)
-					(xy 97.2154 128.656458) (xy 97.352496 128.564134) (xy 97.283843 128.533443) (xy 97.220437 128.489475)
-					(xy 97.161544 128.431266) (xy 97.115033 128.36215) (xy 97.087627 128.286026) (xy 97.078303 128.200334)
-					(xy 97.078974 128.194717) (xy 97.36222 128.194717) (xy 97.366835 128.283383) (xy 97.3806 128.369595)
-					(xy 97.409596 128.444972) (xy 97.45775 128.496967) (xy 97.580207 128.424183) (xy 97.637197 128.382086)
-					(xy 97.674459 128.340752) (xy 97.696467 128.299741) (xy 97.716017 128.230949) (xy 97.722219 128.166751)
-					(xy 97.711213 128.045118) (xy 97.693276 127.995938) (xy 97.662166 127.958412) (xy 97.617998 127.935353)
-					(xy 97.545906 127.926172) (xy 97.468117 127.938363) (xy 97.421098 127.969525) (xy 97.389239 128.017405)
-					(xy 97.372051 128.074427) (xy 97.36222 128.194717) (xy 97.078974 128.194717) (xy 97.089933 128.102989)
-					(xy 97.124344 128.016401) (xy 97.183557 127.937407) (xy 97.23804 127.893616) (xy 97.310514 127.859494)
-					(xy 97.405552 127.836694) (xy 97.528702 127.82823)
-				)
-			)
+					(xy 97.644444 127.835155) (xy 97.724523 127.854714) (xy 97.793172 127.885628) (xy 97.884988 127.952526)
+					(xy 97.956021 128.035226) (xy 98.010277 128.131228) (xy 98.046635 128.231109) (xy 98.067993 128.333838)
+					(xy 98.074738 128.426992) (xy 98.069885 128.479813) (xy 98.052725 128.552899) (xy 98.023576 128.626336)
+					(xy 97.976751 128.70262) (xy 97.915334 128.769435) (xy 97.832388 128.827184) (xy 97.734965 128.863961)
+					(xy 97.607135 128.877498) (xy 97.537552 128.870764) (xy 97.472496 128.850875) (xy 97.340208 128.779556)
+					(xy 97.365736 128.926713) (xy 97.41255 129.064954) (xy 97.478542 129.188151) (xy 97.555737 129.280376)
+					(xy 97.63058 129.340921) (xy 97.706237 129.384271) (xy 97.783448 129.411901) (xy 97.901925 129.436747)
+					(xy 98.008594 129.448293) (xy 98.011051 129.507034) (xy 98.005343 129.538472) (xy 97.993954 129.562965)
+					(xy 97.82626 129.550699) (xy 97.695291 129.528039) (xy 97.574881 129.490895) (xy 97.471214 129.441332)
+					(xy 97.374799 129.376156) (xy 97.278979 129.291612) (xy 97.1945 129.191302) (xy 97.127462 129.077607)
+					(xy 97.077021 128.948817) (xy 97.042033 128.812181) (xy 97.02142 128.677681) (xy 97.014617 128.544473)
+					(xy 97.01507 128.53336) (xy 97.323111 128.53336) (xy 97.323111 128.599061) (xy 97.325569 128.664762)
+					(xy 97.39213 128.707837) (xy 97.436913 128.726434) (xy 97.514063 128.737547) (xy 97.565958 128.730984)
+					(xy 97.609398 128.712269) (xy 97.646244 128.681615) (xy 97.690598 128.619644) (xy 97.722219 128.543129)
+					(xy 97.740626 128.45984) (xy 97.746689 128.376556) (xy 97.739765 128.224894) (xy 97.721867 128.117429)
+					(xy 97.696467 128.043653) (xy 97.657531 127.979975) (xy 97.619368 127.947366) (xy 97.580207 127.937285)
+					(xy 97.520828 127.948707) (xy 97.460208 127.984912) (xy 97.426203 128.021422) (xy 97.393441 128.078108)
+					(xy 97.362327 128.161133) (xy 97.342342 128.248605) (xy 97.328412 128.369819) (xy 97.323111 128.53336)
+					(xy 97.01507 128.53336) (xy 97.020695 128.395273) (xy 97.0373 128.275158) (xy 97.062382 128.17933)
+					(xy 97.099447 128.088854) (xy 97.141987 128.01704) (xy 97.189754 127.961099) (xy 97.273661 127.895972)
+					(xy 97.363503 127.856196) (xy 97.457965 127.835146) (xy 97.550822 127.82823)
+				)
+			)
